File: hackpads/HackPanel/PCB/HackPanel.kicad_pcb (KiCad board)
At the start: 2 copper layers, 77 x 65 mm, 9 parts, among them SW1 RotaryEncoder_Switch, SW3 SW_Push, SW4 SW_Push, SW5 SW_Push, SW6 SW_Push, SW7 SW_Push, U1 XIAO-RP2040-DIP

Commit message: Update HackPanel.kicad_pcb
Other:
- board text added: "HackPanel"
- board text removed: "three_1415"
Changed lines of the file:
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@@
 		)
 	)
-	(gr_text "three_1415"
+	(gr_text "HackPanel"
 		(at 116 123 90)
 		(layer "F.SilkS")
